File: 616_buffer/616_buffer.kicad_pcb (KiCad board)
At the start: 2 copper layers, 52.6 x 43.9 mm, 25 parts, among them J1 1K_Zero, J2 Edge_J104, J3 Air_Pin, U1 LM317L_SO8, U2 LM337L_SO8, U3 LMC6081

Commit message: Fixed zero connector pinout
Connections:
- J1 pad 1: Net-(C6-Pad2) -> Net-(R3-Pad1)
- J1 pad 2: Net-(J1-Pad2) -> Net-(C6-Pad2)
- R3 pad 1: Net-(J1-Pad2) -> Net-(R3-Pad1)
Routing:
- net Net-(R3-Pad1): track 0.00 -> 36.3 mm
- net Net-(J1-Pad2): track 33.9 -> 0.00 mm
- net Net-(C6-Pad2): track 11.2 -> 12.4 mm
Changed lines of the file:
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@@
   (net 8 "Net-(C6-Pad2)")
   (net 9 "Net-(C7-Pad1)")
-  (net 10 "Net-(J1-Pad2)")
+  (net 10 "Net-(R3-Pad1)")
   (net 11 "Net-(J2-Pad1)")
   (net 12 "unconnected-(J2-Pad3)")
@@
     (fp_line (start 8.23 -1.25) (end 1.93 -1.25) (layer "F.Fab") (width 0.1))
     (pad "1" thru_hole circle (at 0 0) (size 1.6 1.6) (drill 0.8) (layers *.Cu *.Mask)
-      (net 10 "Net-(J1-Pad2)") (pintype "passive"))
+      (net 10 "Net-(R3-Pad1)") (pintype "passive"))
     (pad "2" thru_hole oval (at 10.16 0) (size 1.6 1.6) (drill 0.8) (layers *.Cu *.Mask)
       (net 7 "Net-(C5-Pad2)") (pintype "passive"))
@@
     (fp_line (start 1.27 6.35) (end -1.27 6.35) (layer "F.Fab") (width 0.1))
     (pad "1" thru_hole rect (at 0 0 180) (size 1.7 1.7) (drill 1) (layers *.Cu *.Mask)
-      (net 8 "Net-(C6-Pad2)") (pinfunction "Pin_1") (pintype "passive"))
+      (net 10 "Net-(R3-Pad1)") (pinfunction "Pin_1") (pintype "passive"))
     (pad "2" thru_hole oval (at 0 2.54 180) (size 1.7 1.7) (drill 1) (layers *.Cu *.Mask)
-      (net 10 "Net-(J1-Pad2)") (pinfunction "Pin_2") (pintype "passive"))
+      (net 8 "Net-(C6-Pad2)") (pinfunction "Pin_2") (pintype "passive"))
     (pad "3" thru_hole oval (at 0 5.08 180) (size 1.7 1.7) (drill 1) (layers *.Cu *.Mask)
       (net 9 "Net-(C7-Pad1)") (pinfunction "Pin_3") (pintype "passive"))
@@
   (segment (start 147.32 112.522) (end 144.78 112.522) (width 0.4) (layer "F.Cu") (net 7))
   (segment (start 120.396 121.92) (end 122.834 121.92) (width 0.6) (layer "F.Cu") (net 8))
-  (segment (start 114.808 121.92) (end 120.396 121.92) (width 0.6) (layer "F.Cu") (net 8))
+  (segment (start 119.4835 121.5155) (end 120.65 121.5155) (width 0.6) (layer "F.Cu") (net 8))
   (segment (start 123.21 121.544) (end 125.8385 121.544) (width 0.6) (layer "F.Cu") (net 8))
   (segment (start 125.8385 121.544) (end 125.867 121.5155) (width 0.6) (layer "F.Cu") (net 8))
   (segment (start 122.834 121.92) (end 123.21 121.544) (width 0.6) (layer "F.Cu") (net 8))
+  (segment (start 117.348 119.38) (end 119.4835 121.5155) (width 0.6) (layer "F.Cu") (net 8))
+  (segment (start 114.808 119.38) (end 117.348 119.38) (width 0.6) (layer "F.Cu") (net 8))
   (segment (start 117.348 116.078) (end 120.142 116.078) (width 0.6) (layer "F.Cu") (net 9))
   (segment (start 122.814 116.586) (end 122.936 116.464) (width 0.6) (layer "F.Cu") (net 9))
@@
   (segment (start 125.222 116.4355) (end 122.9645 116.4355) (width 0.6) (layer "F.Cu") (net 9))
   (segment (start 116.586 116.84) (end 117.348 116.078) (width 0.6) (layer "F.Cu") (net 9))
-  (segment (start 135.128 108.966) (end 134.874 109.22) (width 0.6) (layer "F.Cu") (net 10))
-  (segment (start 119.888 107.696) (end 134.874 107.696) (width 0.6) (layer "F.Cu") (net 10))
-  (segment (start 112.014 115.57) (end 119.888 107.696) (width 0.6) (layer "F.Cu") (net 10))
-  (segment (start 114.808 119.38) (end 113.03 119.38) (width 0.6) (layer "F.Cu") (net 10))
-  (segment (start 135.128 107.95) (end 135.128 108.966) (width 0.6) (layer "F.Cu") (net 10))
-  (segment (start 112.014 118.364) (end 112.014 115.57) (width 0.6) (layer "F.Cu") (net 10))
-  (segment (start 134.874 107.696) (end 135.128 107.95) (width 0.6) (layer "F.Cu") (net 10))
-  (segment (start 113.03 119.38) (end 112.014 118.364) (width 0.6) (layer "F.Cu") (net 10))
+  (segment (start 135.128 107.95) (end 134.874 107.696) (width 0.6) (layer "F.Cu") (net 10))
+  (segment (start 134.874 107.696) (end 119.888 107.696) (width 0.6) (layer "F.Cu") (net 10))
+  (segment (start 112.014 120.65) (end 113.284 121.92) (width 0.6) (layer "F.Cu") (net 10))
+  (segment (start 113.284 121.92) (end 114.808 121.92) (width 0.6) (layer "F.Cu") (net 10))
+  (segment (start 134.874 109.22) (end 135.128 108.966) (width 0.6) (layer "F.Cu") (net 10))
+  (segment (start 112.014 115.57) (end 112.014 120.65) (width 0.6) (layer "F.Cu") (net 10))
+  (segment (start 135.128 108.966) (end 135.128 107.95) (width 0.6) (layer "F.Cu") (net 10))
+  (segment (start 119.888 107.696) (end 112.014 115.57) (width 0.6) (layer "F.Cu") (net 10))
   (segment (start 157.734 119.126) (end 146.05 135.128) (width 0.6) (layer "F.Cu") (net 11))
   (segment (start 157.861 115.189) (end 157.988 115.316) (width 0.6) (layer "F.Cu") (net 11))
