File: 616_buffer.kicad_pcb (KiCad board)
At the start: 2 copper layers, 52.6 x 43.9 mm, 25 parts, among them J1 1K_Zero, J2 Edge_J104, J3 Air_Pin, U1 LM317L_SO8, U2 LM337L_SO8, U3 LMC6081

Commit message: Update schematic
Parts:
- C5: value 100p -> 2n2
- R3, R5: footprint Resistor_THT:R_Axial_DIN0207_L6.3mm_D2.5mm_P10.16mm_Horizontal -> Resistor_SMD:R_0805_2012Metric
- moved R5 15.5 mm to (144.5, 110.2)
- moved R3 6.20 mm to (141.1, 109.2)
- moved R4 1.37 mm to (145.0, 115.3)
Routing:
- net Net-(C5-Pad2): track 60.4 -> 12.9 mm
- net /C: track 74.5 -> 121.2 mm, vias 0 -> 2
- net Net-(J1-Pad1): track 36.3 -> 39.2 mm
- net Net-(J3-Pad1): track 4.39 -> 3.02 mm
- net Net-(R4-Pad2): track 3.17 -> 4.54 mm
Other:
- board text added: "1"
- board text added: "6"
